File: STM32_UART_board/STM32_UART_board.kicad_sch (KiCad schematic)
At the start: 24 parts, among them J1 SWD, J2 Scooter, J3 Conn_01x10, J4 Conn_01x10, Q1 AO4612_C4748739, SW1 SW_Push, U1 BAS70-05, U2 LM2574HVM-5, U3 AMS1117-3.3, U4 STM32C011F6Px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

Commit message: component placemnt 15%
Parts:
- removed C4: 100 uF, symbol Device:C_Polarized
- removed J4: Conn_01x10, Connector_PinHeader_2.54mm:PinHeader_1x10_P2.54mm_Vertical, symbol Connector_Generic:Conn_01x10
- removed U3: AMS1117-3.3, Package_TO_SOT_SMD:SOT-223-3_TabPin2, symbol Regulator_Linear:AMS1117-3.3
- added C4, C5: 22u|10V, Capacitor_SMD:C_0805_2012Metric_Pad1.18x1.45mm_HandSolder, symbol Device:C
- added C6: 100n|50V, Capacitor_SMD:C_0603_1608Metric_Pad1.08x0.95mm_HandSolder, symbol Device:C_Small
- added C7: 4.7u, Capacitor_SMD:C_0805_2012Metric_Pad1.18x1.45mm_HandSolder, symbol Device:C
- added C9: 100n, Capacitor_SMD:C_0603_1608Metric_Pad1.08x0.95mm_HandSolder, symbol Device:C
- added D2: LED, LED_SMD:LED_0805_2012Metric_Pad1.15x1.40mm_HandSolder, symbol Device:LED
- added R4, R5, R6: 100k, Resistor_SMD:R_0603_1608Metric_Pad0.98x0.95mm_HandSolder, symbol Device:R
- added SW2: SW_Push, Button_Switch_THT:SW_PUSH_6mm, symbol Switch:SW_Push
- added U3: AZ1117-3.3, Package_TO_SOT_SMD:SOT-223-3_TabPin2, symbol Regulator_Linear:AZ1117-3.3
- C1: footprint (none) -> Capacitor_SMD:CP_Elec_6.3x7.7; Shop (none) -> https://www.tme.eu/pl/details/gsc00bm2201jarl/kondensatory-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
- C3: footprint (none) -> Capacitor_SMD:CP_Elec_8x10
- D1: value 1N5819 -> SK26; footprint (none) -> Diode_SMD:D_SMB_Handsoldering; Shop (none) -> https://www.tme.eu/pl/en/details/sk26-dio/smd-schottky-diod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
- J2: footprint Connector_PinSocket_1.27mm:PinSocket_1x05_P1.27mm_Vertical -> Connector_Molex:Molex_Micro-Latch_53253-0570_1x05_P2.00mm_Vertical
- J3: now not fitted; now left out of the parts list
- L1: value 330 uH -> 680 uH; footprint Inductor_SMD:L_7.3x7.3_H4.5 -> Inductor_SMD:L_12x12mm_H8mm
- Q1: Shop (none) -> https://www.tme.eu/pl/details/ao4611/tranzystory-multikanal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
- R1, R2, R3: footprint (none) -> Resistor_SMD:R_0603_1608Metric_Pad0.98x0.95mm_HandSolder
- SW1: footprint (none) -> Button_Switch_THT:SW_PUSH_6mm
- U1: Shop (none) -> https://www.tme.eu/pl/en/details/bas70-05-dio/smd-schottky-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
Connections:
- net PIN_13 is gone; now on net BUTTON: U4.13 (PA6)
- net PIN_14 is gone; now on net EN: U4.14 (PA7)
- net VCC is gone; now on net BATT+: J2.1 (Pin_1)
- net +3.3V: now also C5.1, C6.1, C7.1, C9.1, R5.1, SW2.2, U3.2 (VO)
- net +5V: now also C4.1, U3.3 (VI)
- net BUTTON: now also R5.2; no longer U4.16 (PA9/PA11)
- net EN: no longer U4.17 (PA10/PA12), U5.6 (PA10/PA12)
- net GND: now also C4.2, C5.2, C6.2, C7.2, C9.2, D2.1 (K), R6.2, U3.1 (GND)
- net NRST: no longer J3.6 (Pin_6)
- net PIN_01: no longer U4.1 (PB7)
- net PIN_02: no longer J2.3 (Pin_3), U4.2 (PC14)
- net PIN_03: no longer U4.3 (PC15)
- net PIN_07: no longer U4.7 (PA0)
- net PIN_08: no longer U4.8 (PA1)
- net PIN_09: no longer U4.9 (PA2)
- net PIN_10: no longer U4.10 (PA3)
- net PIN_15: no longer Q1.2 (G2), R3.1, U4.15 (PA8)
- net PIN_18: no longer J1.3 (Pin_3), U4.18 (PA13)
- net PIN_11 renamed PA4
- net PIN_12 renamed ON
- net ON: now also Q1.2 (G2), R3.1
- net PIN_19 renamed PA14
- net PIN_20 renamed PB6
- new net: D2.2 (A), R4.2
- new net BOOT0_USART1_RX: U4.17 (PA10/PA12)
- new net BOOT0_USART1_TX: U4.16 (PA9/PA11)
- new net PA0: U4.7 (PA0)
- new net PA1: R6.1, SW2.1, U4.8 (PA1)
- new net PA13: J1.3 (Pin_3), U4.18 (PA13)
- new net PA2: U4.9 (PA2)
- new net PA3: U4.10 (PA3)
- new net PA8: R4.1, U4.15 (PA8)
- new net PB7: U4.1 (PB7)
- new net PC14: J2.3 (Pin_3), U4.2 (PC14)
- new net PC15: U4.3 (PC15)
- new net PIN_06: J3.6 (Pin_6)
- new net PIN_17: U5.6 (PA10/PA12)
- no-connect marks 0 -> 1
Other:
- note added: "100nF for evey VDD 4.7uF at common point"
- note added: "Decoupling"
- note added: "User interface and buckup"
- note added: "enable internal pullup or populate R5"
