File: STM32_UART_board/STM32_UART_board.kicad_pcb (KiCad board)
At the start: 2 copper layers, 30 parts, among them J1 SWD, J2 Scooter, Q1 AO4612_C4748739, SW1 SW_Push, SW2 SW_Push, U1 BAS70-05, U2 LM2574HVM-5, U3 AZ1117-3.3, U4 STM32C011F6Px

Commit message: component placement 16%
Parts:
- moved U4 12.5 mm to (96.0, 174.5)
Changed lines of the file:
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@@
 	(footprint "Package_SO:TSSOP-20_4.4x6.5mm_P0.65mm"
 		(layer "F.Cu")
-		(at 107.5875 169.775)
+		(at 96 174.5)
 		(descr "TSSOP, 20 Pin (JEDEC MO-153 Var AC https://www.jedec.org/document_search?search_api_views_fulltext=MO-153), generated with kicad-footprint-generator ipc_gullwing_generator.py")
 		(tags "TSSOP SO")
